File: usb2ps2.kicad_pcb (KiCad board)
At the start: 2 copper layers, 49.5 x 26 mm, 24 parts, among them CN1 Conn_01x02, CN2 UART, CN3 PS/2 Pins

Commit message: HW Rev 1.0 minor updates
Routing:
- net /GPIO14: track 94.6 -> 95.2 mm
- net /PS2 with Diodes/KB_DATA: track 18.4 -> 17.7 mm
- net GND: vias 18 -> 19
